Commit message: commit

File: robots/uw_assembly_auv_sensors.xacro (robot description, xacro)
@@ -21,5 +21,5 @@
   </xacro:default_imu_macro>
   <xacro:fisheye_camera namespace="${namespace}" parent_link="${namespace}/base_link" suffix="">
-	  <origin xyz="0.01 2.0 0.75" rpy="0 1.57 0"/>
+	  <origin xyz="-2.51 0.0 1.75" rpy="0 1.57 0"/>
   </xacro:fisheye_camera>
   <xacro:default_pose_3d_macro
